File: .kicad_sch (KiCad schematic)
At the start: 0 parts

Commit message: Commit vor PCB Layout
Other:
- sheet KomModul_TragFluegel renamed Stammblatt
- sheet Stammblatt: file KomModul_TragFluegel.kicad_sch -> KomModul_Joystick.kicad_sch
Changed lines of the file:
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@@
 			(color 0 0 0 0)
 		)
-		(property "Sheetname" "KomModul_TragFluegel"
+		(property "Sheetname" "Stammblatt"
 			(at 0 -0.7116 0)
 			(show_name no)
@@
 			)
 		)
-		(property "Sheetfile" "KomModul_TragFluegel.kicad_sch"
+		(property "Sheetfile" "KomModul_Joystick.kicad_sch"
 			(at 0 4.3946 0)
 			(show_name no)
