File: KomModul_TragFluegel.kicad_pcb (KiCad board)
At the start: 2 copper layers, 100 x 100 mm, 61 parts, among them J1 MotorA, J2 MotorB, J3 JTAG, J4 SPI, J5 Joystick, J6 Reserve_Klemme, J7 I2C/RTC, J8 ISP, Q1 BC547, Q2 BC546, SW1 Wahlschalter_Supply, SW2 Reset, U1 ATmega1284P-PU, U2 MAX485E_A, U3 MAX485E_B, U4 MCP23017_SP, U5 4 X 20 Textdisplay, Y1 16MHz

Commit message: Commit new PCB Layout
Parts:
- removed D1, D3: LEDVers, LED_THT:LED_D5.0mm
- removed D2, D4: D, Resistor_THT:R_Axial_DIN0207_L6.3mm_D2.5mm_P10.16mm_Horizontal
- removed D7: Z_5.1V, Resistor_THT:R_Axial_DIN0207_L6.3mm_D2.5mm_P10.16mm_Horizontal
- removed D8: 1N4936, Resistor_THT:R_Axial_DIN0207_L6.3mm_D2.5mm_P10.16mm_Horizontal
- removed F1: F250mA, MyLib:Schurter_horizontal_3101.0055
- removed J7: I2C/RTC, TerminalBlock_TE-Connectivity:TerminalBlock_TE_282834-5_1x05_P2.54mm_Horizontal
- removed J8: ISP, Connector_Dsub:DSUB-9_Female_Horizontal_P2.77x2.84mm_EdgePinOffset4.94mm_Housed_MountingHolesOffset7.48mm
- removed L1: 10µH, Resistor_THT:R_Axial_DIN0309_L9.0mm_D3.2mm_P12.70mm_Horizontal
- removed Q1: BC547, Package_TO_SOT_THT:TO-92_Inline
- removed Q2: BC546, Package_TO_SOT_THT:TO-92_Inline
- removed R14, R16, R19: 10k, Resistor_THT:R_Axial_DIN0207_L6.3mm_D2.5mm_P10.16mm_Horizontal
- removed R15, R17: 4.7k, Resistor_THT:R_Axial_DIN0207_L6.3mm_D2.5mm_P10.16mm_Horizontal
- removed R18: 33k, Resistor_THT:R_Axial_DIN0207_L6.3mm_D2.5mm_P10.16mm_Horizontal
- removed R20: 300, Resistor_THT:R_Axial_DIN0207_L6.3mm_D2.5mm_P10.16mm_Horizontal
- removed SW2: Reset, Button_Switch_THT:SW_PUSH_6mm_H4.3mm
- removed U5: 4 X 20 Textdisplay, Connector_IDC:IDC-Header_2x08_P2.54mm_Horizontal
- added C15: 10 nF, Capacitor_SMD_Wurth:C_Wurth_WCAP-CSGP-1206_H0.8, F.Cu at (151.4, 76.5)
- added C16: 1 uF, Capacitor_SMD_Wurth:C_Wurth_WCAP-CSGP-1206_H1.15, F.Cu at (151.4, 79.8)
- added C17: 22 pF, Capacitor_SMD_Wurth:C_Wurth_WCAP-CSGP-1206_H0.8, F.Cu at (151.4, 83.0)
- added C18: 22 pF, Capacitor_SMD_Wurth:C_Wurth_WCAP-CSGP-1206_H0.8, F.Cu at (151.4, 86.2)
- added R2: 120 ohm, Resistor_SMD_Wurth:R_Wurth_WRIS-RSKS-1210_R, F.Cu at (123.0, 94.9)
- added SW3: 472123010111, Switch_THT_Wurth:SW_Wurth_WS-TOTV_472123010111, F.Cu at (108.5, 96.8)
- C1: value 330µF -> 10 nF; footprint Capacitor_THT:CP_Radial_D12.5mm_P5.00mm -> Capacitor_SMD_Wurth:C_Wurth_WCAP-CSGP-1206_H0.8
- C10, C13: value 100nF -> 100 nF; footprint Capacitor_THT:C_Disc_D5.0mm_W2.5mm_P2.50mm -> Capacitor_SMD_Wurth:C_Wurth_WCAP-CSGP-1206_H0.8
- C11: value 100nF -> 100 uF; footprint Capacitor_THT:C_Disc_D5.0mm_W2.5mm_P2.50mm -> Capacitor_THT_Wurth:CP_Wurth_WCAP-PT5H-P2.5D6.3L11
- C12: value 100nF -> 10 uF; footprint Capacitor_THT:C_Disc_D5.0mm_W2.5mm_P2.50mm -> Capacitor_SMD_Wurth:C_Wurth_WCAP-CSGP-1206_H1.6
- C14: value 100nF -> 4.7 uF; footprint Capacitor_THT:C_Disc_D5.0mm_W2.5mm_P2.50mm -> Capacitor_SMD_Wurth:C_Wurth_WCAP-CSGP-1206_H1.6
- C2: value 470nF -> 10 nF; footprint Capacitor_THT:C_Disc_D7.5mm_W5.0mm_P10.00mm -> Capacitor_SMD_Wurth:C_Wurth_WCAP-CSGP-1206_H0.8
- C3: value 100nF -> 10 nF; footprint Capacitor_THT:C_Disc_D5.0mm_W2.5mm_P2.50mm -> Capacitor_SMD_Wurth:C_Wurth_WCAP-CSGP-1206_H0.8
- C4, C5: value 22pF -> 100 nF; footprint Capacitor_THT:C_Disc_D5.0mm_W2.5mm_P2.50mm -> Capacitor_SMD_Wurth:C_Wurth_WCAP-CSGP-0805_H0.8_R
- C6, C7: value 100nF -> 1 uF; footprint Capacitor_THT:C_Disc_D5.0mm_W2.5mm_P2.50mm -> Capacitor_SMD_Wurth:C_Wurth_WCAP-CSGP-1206_H1.15
- C8: value 330µF -> 100 nF; footprint Capacitor_THT:CP_Radial_D12.5mm_P5.00mm -> Capacitor_SMD_Wurth:C_Wurth_WCAP-CSGP-1206_H0.8
- C9: value 470nF -> 100 nF; footprint Capacitor_THT:C_Disc_D7.5mm_W5.0mm_P10.00mm -> Capacitor_SMD_Wurth:C_Wurth_WCAP-CSGP-1206_H0.8
- D5: value LED_SPI -> 5mmWOS_151051RS11000; footprint LED_THT:LED_D5.0mm -> LED_THT_Wurth:D_Wurth_WL-TMRC-5mmWOS
- D6: value Z_5.1V -> 5mmWOS_151051RS11000; footprint Resistor_THT:R_Axial_DIN0207_L6.3mm_D2.5mm_P10.16mm_Horizontal -> LED_THT_Wurth:D_Wurth_WL-TMRC-5mmWOS
- J1: value MotorA -> 66100411622; footprint MyLib:TerminalBlock_RND_01.04_P_3.50mm -> Connector_THT_Wurth:J_Wurth_WR-WTB_66100411622
- J2: value MotorB -> 618015231121; footprint MyLib:TerminalBlock_RND_01.04_P_3.50mm -> Connector_THT_Wurth:J_Wurth_WR-DSUB_618015231121
- J3: value JTAG -> 691242510004; footprint Connector_IDC:IDC-Header_2x05_P2.54mm_Vertical -> Terminal_Wuerth_Block:691242510004
- J4: value SPI -> 691242510004; footprint Connector_IDC:IDC-Header_2x03_P2.54mm_Vertical -> Terminal_Wuerth_Block:691242510004
- J5: value Joystick -> 612020235121; footprint Connector_Dsub:DSUB-15_Female_Horizontal_P2.77x2.84mm_EdgePinOffset4.94mm_Housed_MountingHolesOffset7.48mm -> Connector_THT_Wurth:J_Wurth_WR-BHD_612020235121
- J6: value Reserve_Klemme -> 696106003002; footprint TerminalBlock_TE-Connectivity:TerminalBlock_TE_1-282834-0_1x10_P2.54mm_Horizontal -> Connector_THT_Wurth:J_Wurth_WR-FSH_696106003002
- R1: value 230 -> 4.7 kohm; footprint Resistor_THT:R_Axial_DIN0207_L6.3mm_D2.5mm_P10.16mm_Horizontal -> Resistor_SMD_Wurth:R_Wurth_WRIS-RSKS-1206_R
- R10: value 15k -> 8.2 kohm; footprint Resistor_THT:R_Axial_DIN0207_L6.3mm_D2.5mm_P10.16mm_Horizontal -> Resistor_SMD_Wurth:R_Wurth_WRIS-RSKS-1206_R
- R11: value 47R -> 10 kohm; footprint Resistor_THT:R_Axial_DIN0207_L6.3mm_D2.5mm_P10.16mm_Horizontal -> Resistor_SMD_Wurth:R_Wurth_WRIS-RSKS-1206_R
- R12: value 4,3k -> 10 kohm; footprint Resistor_THT:R_Axial_DIN0207_L6.3mm_D2.5mm_P10.16mm_Horizontal -> Resistor_SMD_Wurth:R_Wurth_WRIS-RSKS-1206_R
- R13: value 10k -> 10 kohm; footprint Resistor_THT:R_Axial_DIN0207_L6.3mm_D2.5mm_P10.16mm_Horizontal -> Resistor_SMD_Wurth:R_Wurth_WRIS-RSKS-1206_R
- R3: value 230 -> 8.2 kohm; footprint Resistor_THT:R_Axial_DIN0207_L6.3mm_D2.5mm_P10.16mm_Horizontal -> Resistor_SMD_Wurth:R_Wurth_WRIS-RSKS-1206_R
- R4: value 10M -> 4.7 kohm; footprint Resistor_THT:R_Axial_DIN0207_L6.3mm_D2.5mm_P10.16mm_Horizontal -> Resistor_SMD_Wurth:R_Wurth_WRIS-RSKS-1206_R
- R5: value 60 -> 120 ohm; footprint Resistor_THT:R_Axial_DIN0207_L6.3mm_D2.5mm_P10.16mm_Horizontal -> Resistor_SMD_Wurth:R_Wurth_WRIS-RSKS-1210_R
- R6: value 60 -> 1 kohm; footprint Resistor_THT:R_Axial_DIN0207_L6.3mm_D2.5mm_P10.16mm_Horizontal -> Resistor_SMD_Wurth:R_Wurth_WRIS-RSKS-1206_R
- R7: value 5,6k -> 1 kohm; footprint Resistor_THT:R_Axial_DIN0207_L6.3mm_D2.5mm_P10.16mm_Horizontal -> Resistor_SMD_Wurth:R_Wurth_WRIS-RSKS-1206_R
- R8: value 5,6k -> 8.2 kohm; footprint Resistor_THT:R_Axial_DIN0207_L6.3mm_D2.5mm_P10.16mm_Horizontal -> Resistor_SMD_Wurth:R_Wurth_WRIS-RSKS-1206_R
- R9: value 5k -> 4.7 kohm; footprint Potentiometer_THT:Potentiometer_Piher_PT-6-V_Vertical -> Resistor_SMD_Wurth:R_Wurth_WRIS-RSKS-1206_R
- SW1: value Wahlschalter_Supply -> 430182080816; footprint Button_Switch_THT:SW_DIP_SPSTx03_Slide_6.7x9.18mm_W7.62mm_P2.54mm_LowProfile -> Switch_SMD_Wurth:SW_Wurth_WS-TASV_430182080816
- U1: value ATmega1284P-PU -> STM32F303RETx; footprint Package_DIP:DIP-40_W15.24mm -> Package_QFP:LQFP-64_10x10mm_P0.5mm
- U2: value MAX485E_A -> SP3485EN; footprint Package_DIP:DIP-8_W7.62mm_Socket -> Package_SO:SOIC-8_3.9x4.9mm_P1.27mm
- U3: value MAX485E_B -> SP3485EN; footprint Package_DIP:DIP-8_W7.62mm_Socket -> Package_SO:SOIC-8_3.9x4.9mm_P1.27mm
- U4: value MCP23017_SP -> TLV1117LV33DCYR; footprint Package_DIP:DIP-28_W7.62mm_LongPads -> MyLib:VREG_TLV1117LV33DCYR
- Y1: value 16MHz -> 16 MHz; footprint Crystal:Crystal_HC49-4H_Vertical -> Crystal_THT_Wurth:Y_Wurth_WE-XTAL_Quartz-HC49-4H
- moved D6 88.6 mm to (162.5, 48.2), turned to 0 degrees
- moved J4 85.6 mm to (148.6, 54.5), turned to 0 degrees
- moved J3 81.0 mm to (148.6, 43.0), turned to 0 degrees
- moved D5 80.9 mm to (162.5, 40.7), turned to 0 degrees
- moved C5 68.4 mm to (161.7, 56.3), turned to 0 degrees
- moved J1 65.0 mm to (148.4, 91.4), turned to 0 degrees
- moved R11 64.1 mm to (134.6, 80.2), turned to 0 degrees
- moved J5 64.0 mm to (130.8, 43.1), turned to 0 degrees
- moved C4 63.8 mm to (161.7, 53.4), turned to 0 degrees
- moved R7 61.8 mm to (129.2, 86.6), turned to 0 degrees
- moved R8 57.4 mm to (129.2, 89.9), turned to 0 degrees
- moved R9 46.7 mm to (134.6, 73.7), turned to 0 degrees
- moved C11 45.1 mm to (161.2, 92.0), turned to 0 degrees
- moved C13 45.0 mm to (145.9, 86.2)
- moved Y1 44.3 mm to (158.2, 74.8), turned to 0 degrees
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Connections:
- C1 pad 1: Net-(C1-Pad1) -> /JS_X_axis
- C10 pad 1: Net-(C10-Pad1) -> GND
- C10 pad 2: GND -> /VCC_3_3V
- C11 pad 1: /VCC -> /VCC_5V
- C12 pad 1: /VCC -> GND
- C12 pad 2: GND -> /VCC_5V
- C13 pad 2: /VCC -> /VCC_3_3V
- C14 pad 1: Net-(C14-Pad1) -> /VCC_3_3V
- C2 pad 1: Net-(C1-Pad1) -> GND
- C2 pad 2: GND -> /JS_Z_axis
- C3 pad 1: Net-(C1-Pad1) -> /JS_Y_axis
- C4 pad 1: Net-(C4-Pad1) -> GND
- C4 pad 2: GND -> /VCC_3_3V
- C5 pad 1: Net-(C5-Pad1) -> GND
- C5 pad 2: GND -> /VCC_3_3V
- C6 pad 1: /VCC -> /VCC_3_3V
- C7 pad 1: GND -> /VCC_5V
- C7 pad 2: Net-(C7-Pad2) -> GND
- C8 pad 1: Net-(C10-Pad1) -> GND
- C8 pad 2: GND -> /VCC_3_3V
- C9 pad 1: Net-(C10-Pad1) -> /VCC_3_3V
- D5 pad 1: Net-(D5-Pad1) -> Net-(D5-+)
- D5 pad 2: Net-(D5-Pad2) -> GND
- D6 pad 1: /SCK -> Net-(D6-+)
- J1 pad 1: Net-(C1-Pad1) -> GND
- J1 pad 2: GND -> /VCC_3_3V
- J1 pad 3: /RS485A_A -> /Display_SDA
- J1 pad 4: /RS485B_A -> /Display_SCL
- J2 pad 1: Net-(C10-Pad1) -> Net-(J2-Pad1)
- J2 pad 2: GND -> Net-(J2-Pad2)
- J2 pad 3: /RS485A_B -> unconnected-(J2-Pad3)
- J2 pad 4: /RS485B_B -> GND
- J3 pad 1: /TCK -> /RS485_B_Mtr_A
- J3 pad 2: GND -> /RS485_A_Mtr_A
- J3 pad 3: /TDO -> GND
- J3 pad 4: /VCC -> Net-(J3-Pad4)
- J4 pad 1: /VCC -> /RS485_B_Mtr_B
- J4 pad 2: /~{SS_EXT} -> /RS485_A_Mtr_B
- J4 pad 3: /MOSI -> GND
- J4 pad 4: /MISO -> Net-(J4-Pad4)
- J5 pad 1: /JY_Sig -> /VCC_3_3V
- J5 pad 10: /JT2 -> GND
- J5 pad 11: Net-(J5-Pad11) -> unconnected-(J5-Pad11)
- J5 pad 12: Net-(J5-Pad12) -> GND
- J5 pad 13: /JT1 -> /SWO
- J5 pad 14: Net-(J5-Pad14) -> GND
- J5 pad 15: Net-(J5-Pad15) -> /NRST
- J5 pad 2: /JX_Sig -> /VCC_3_3V
- J5 pad 6: /VCC -> GND
- J5 pad 7: /VCC -> /SWDIO
- J5 pad 8: /VCC -> GND
- J5 pad 9: /JZ_Sig -> /SWCLK
- J6 pad 1: /VCC -> Net-(J6-Pad1)
- J6 pad 2: /PC6 -> /VCC_5V
- R1 pad 1: Net-(C1-Pad1) -> Net-(J2-Pad1)
- R1 pad 2: Net-(D1-Pad2) -> /JS_X_axis
- R10 pad 1: /VCC -> /JS_Y_axis
- R10 pad 2: Net-(R10-Pad2) -> GND
- R11 pad 1: Net-(R11-Pad1) -> /JS_Taster2
- R11 pad 2: /VCC -> GND
- R12 pad 1: Net-(Q1-Pad2) -> /JS_Taster1
- R12 pad 2: /LEDSPI_en -> GND
- R13 pad 1: GND -> Net-(U1-BOOT0)
- R13 pad 2: /JT1 -> GND
- R3 pad 1: Net-(C10-Pad1) -> /JS_X_axis
- R3 pad 2: Net-(D3-Pad2) -> GND
- R4 pad 1: GND -> Net-(J2-Pad2)
- R4 pad 2: Net-(R4-Pad2) -> /JS_Z_axis
- R5 pad 1: /RS485B_A -> /RS485_A_Mtr_B
- R5 pad 2: /RS485A_A -> /RS485_B_Mtr_B
- R6 pad 1: /RS485B_B -> Net-(J3-Pad4)
- R6 pad 2: /RS485A_B -> Net-(D5-+)
- R7 pad 1: /SCL -> Net-(J4-Pad4)
- R7 pad 2: /VCC -> Net-(D6-+)
- R8 pad 1: /SDA -> /JS_Z_axis
- R8 pad 2: /VCC -> GND
- R9 pad 1: GND -> Net-(J2-Pad9)
- R9 pad 2: Net-(R9-Pad2) -> /JS_Y_axis
- SW1 pad 1: Net-(C1-Pad1) -> /NRST
- SW1 pad 2: Net-(R4-Pad2) -> unconnected-(SW1-Pad2)
- SW1 pad 3: Net-(C10-Pad1) -> unconnected-(SW1-Pad3)
- SW1 pad 4: Net-(F1-Pad2) -> GND
- U1 pad 1: /JT1 -> /VCC_3_3V
- U1 pad 10: /VCC -> unconnected-(U1-PC2-Pad10)
- U1 pad 11: GND -> unconnected-(U1-PC3-Pad11)
- U1 pad 12: Net-(C4-Pad1) -> GND
- U1 pad 13: Net-(C5-Pad1) -> /VCC_3_3V
- U1 pad 14: /RXD_0_A -> unconnected-(U1-PA0-Pad14)
- U1 pad 15: /TXD_0_A -> unconnected-(U1-PA1-Pad15)
- U1 pad 16: /RXD_1_B -> unconnected-(U1-PA2-Pad16)
- U1 pad 17: /TXD_1_B -> unconnected-(U1-PA3-Pad17)
- U1 pad 18: /~{RE_A} -> GND
- U1 pad 19: /DE_A -> /VCC_3_3V
- U1 pad 2: /JT2 -> unconnected-(U1-PC13-Pad2)
- U1 pad 20: /~{RE_B} -> unconnected-(U1-PA4-Pad20)
- U1 pad 21: /DE_B -> unconnected-(U1-PA5-Pad21)
- U1 pad 22: /SCL -> /UART_DE_Mtr_A
- U1 pad 23: /SDA -> /UART_NRE_Mtr_A
- U1 pad 24: /TCK -> /UART_TX_Mtr_A
- U1 pad 25: /TMS -> /UART_RX_Mtr_A
- U1 pad 26: /TDO -> unconnected-(U1-PB0-Pad26)
- U1 pad 27: /TDI -> /UART_DE_Mtr_B
- U1 pad 28: /PC6 -> /UART_NRE_Mtr_B
- U1 pad 29: /PC7 -> /UART_TX_Mtr_B
- U1 pad 3: /PB2_INT2 -> unconnected-(U1-PC14-Pad3)
- U1 pad 30: Net-(C7-Pad2) -> /UART_RX_Mtr_B
- U1 pad 32: Net-(C14-Pad1) -> /VCC_3_3V
- U1 pad 33: /PA_ADC7 -> /JS_X_axis
- U1 pad 34: /PA_ADC6 -> /JS_Taster1
- U1 pad 35: /PA_ADC5 -> /JS_Y_axis
- U1 pad 36: /PA_ADC4 -> /JS_Z_axis
- U1 pad 37: /PA_ADC3 -> /JS_Taster2
- U1 pad 38: /JZ_Sig -> unconnected-(U1-PC7-Pad38)
- U1 pad 39: /JY_Sig -> unconnected-(U1-PC8-Pad39)
- U1 pad 4: /LEDSPI_en -> unconnected-(U1-PC15-Pad4)
- U1 pad 40: /JX_Sig -> unconnected-(U1-PC9-Pad40)
- U1 pad 5: /~{SS_EXT} -> Net-(U1-PF0)
- U1 pad 6: /MOSI -> Net-(U1-PF1)
- U1 pad 7: /MISO -> /NRST
- U1 pad 8: /SCK -> unconnected-(U1-PC0-Pad8)
- U1 pad 9: /~{RESET} -> unconnected-(U1-PC1-Pad9)
- U2 pad 1: /RXD_0_A -> /UART_RX_Mtr_A
- U2 pad 2: /~{RE_A} -> /UART_NRE_Mtr_A
- U2 pad 3: /DE_A -> /UART_DE_Mtr_A
- U2 pad 4: /TXD_0_A -> /UART_TX_Mtr_A
- U2 pad 6: /RS485A_A -> /RS485_A_Mtr_A
- U2 pad 7: /RS485B_A -> /RS485_B_Mtr_A
- U2 pad 8: /VCC -> /VCC_3_3V
- U3 pad 1: /RXD_1_B -> /UART_RX_Mtr_B
- U3 pad 2: /~{RE_B} -> /UART_NRE_Mtr_B
- U3 pad 3: /DE_B -> /UART_DE_Mtr_B
- U3 pad 4: /TXD_1_B -> /UART_TX_Mtr_B
- U3 pad 6: /RS485A_B -> /RS485_A_Mtr_B
- U3 pad 7: /RS485B_B -> /RS485_B_Mtr_B
- U3 pad 8: /VCC -> /VCC_3_3V
- U4 pad 1: Net-(U4-Pad1) -> GND
- U4 pad 2: Net-(U4-Pad2) -> /VCC_3_3V
- U4 pad 3: Net-(U4-Pad3) -> /VCC_5V
- U4 pad 4: Net-(U4-Pad4) -> /VCC_3_3V
- Y1 pad 1: Net-(C4-Pad1) -> Net-(U1-PF0)
- Y1 pad 2: Net-(C5-Pad1) -> Net-(U1-PF1)
Routing:
- net GND: track 549.2 -> 0.00 mm
- net /VCC: track 405.8 -> 0.00 mm
- net /~{RESET}: track 152.4 -> 0.00 mm
- net /MOSI: track 100.5 -> 0.00 mm
- net /MISO: track 80.0 -> 0.00 mm
- net /SCK: track 79.3 -> 0.00 mm
- net /PC6: track 74.7 -> 0.00 mm
- net /PC7: track 74.7 -> 0.00 mm
- net /PB2_INT2: track 68.8 -> 0.00 mm
- net /JT1: track 66.5 -> 0.00 mm
- net Net-(C10-Pad1): track 60.4 -> 0.00 mm
- net /~{SS_EXT}: track 58.0 -> 0.00 mm
- net /JT2: track 57.8 -> 0.00 mm
- net /PA_ADC7: track 50.8 -> 0.00 mm
- net Net-(C1-Pad1): track 49.7 -> 0.00 mm
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- removed copper zone on B.Cu, net GND
- removed copper zone on F.Cu, net GND
Other:
- board outline removed
- board text removed: "Display"
- board text removed: "Display Kontrast"
- board text removed: "FUSE F350mA"
- board text removed: "GND"
- board text removed: "GND R"
- board text removed: "I2C/RTC"
- board text removed: "ISP Progr."
- board text removed: "JTAG"
- board text removed: "Joystick Anschluss"
- board text removed: "Kommunikationsmodul Tragflügelboot Florian Walter"
- board text removed: "M_A"
- board text removed: "M_B"
- board text removed: "Motor A"
- board text removed: "Motor B"
- board text removed: "PA_ADC3"
- board text removed: "PA_ADC4"
- board text removed: "PA_ADC5"
- board text removed: "PA_ADC6"
- board text removed: "PA_ADC7"
- board text removed: "PB_INT2"
- board text removed: "PC6"
- board text removed: "PC7"
- board text removed: "Reserve"
- board text removed: "SPI-Verbindung Master/Slave"
- board text removed: "VCC"
- board text removed: "~{RESET}"
