File: KiCAD_Schaltplan/KommModul_Joystick/KommModul_Joystick.kicad_sch (KiCad schematic)
At the start: 46 parts, among them J1 66100411622, J2 618015231121, J3 691242510004, J4 691242510004, J5 612020235121, J6 696106003002, SW1 430182080816, SW3 472123010111, U1 STM32F303RETx, U2 SP3485EN, U3 SP3485EN, U4 TLV1117LV33DCYR, Y1 16 MHz

Commit message: Manyak Maxim
Whääää
Other:
- note added: "Maxim der Manyak"
Changed lines of the file:
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@@
+		)
+	)
+	(text "Maxim der Manyak"
+		(exclude_from_sim no)
+		(at 258.318 91.948 0)
+		(effects
+			(font
+				(size 1.27 1.27)
+			)
 		)
 	)

Commit message: update schaltplan
Connections:
- no-connect marks 10 -> 41
Other:
- note removed: "Maxim der Manyak"
Changed lines of the file:
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@@
-		)
-	)
-	(text "Maxim der Manyak"
-		(exclude_from_sim no)
-		(at 258.318 91.948 0)
-		(effects
-			(font
-				(size 1.27 1.27)
-			)
 		)
 	)
@@
 	)
 	(no_connect
+		(at 194.31 147.32)
+	)
+	(no_connect
+		(at 173.99 147.32)
+	)
+	(no_connect
+		(at 189.23 111.76)
+	)
+	(no_connect
+		(at 153.67 111.76)
+	)
+	(no_connect
+		(at 161.29 111.76)
+	)
+	(no_connect
+		(at 176.53 147.32)
+	)
+	(no_connect
+		(at 212.09 147.32)
+	)
+	(no_connect
 		(at 182.88 49.53)
 	)
 	(no_connect
+		(at 201.93 147.32)
+	)
+	(no_connect
+		(at 151.13 111.76)
+	)
+	(no_connect
+		(at 207.01 111.76)
+	)
+	(no_connect
+		(at 176.53 111.76)
+	)
+	(no_connect
+		(at 168.91 147.32)
+	)
+	(no_connect
+		(at 179.07 111.76)
+	)
+	(no_connect
+		(at 158.75 111.76)
+	)
+	(no_connect
+		(at 217.17 111.76)
+	)
+	(no_connect
+		(at 163.83 111.76)
+	)
+	(no_connect
+		(at 214.63 111.76)
+	)
+	(no_connect
 		(at 182.88 69.85)
 	)
 	(no_connect
+		(at 204.47 147.32)
+	)
+	(no_connect
 		(at 182.88 64.77)
 	)
 	(no_connect
+		(at 209.55 147.32)
+	)
+	(no_connect
+		(at 171.45 111.76)
+	)
+	(no_connect
 		(at 243.84 63.5)
 	)
 	(no_connect
+		(at 156.21 111.76)
+	)
+	(no_connect
+		(at 196.85 147.32)
+	)
+	(no_connect
+		(at 204.47 111.76)
+	)
+	(no_connect
 		(at 182.88 54.61)
 	)
 	(no_connect
+		(at 181.61 147.32)
+	)
+	(no_connect
 		(at 243.84 55.88)
 	)
 	(no_connect
+		(at 173.99 111.76)
+	)
+	(no_connect
 		(at 243.84 66.04)
 	)
@@
 	)
 	(no_connect
+		(at 207.01 147.32)
+	)
+	(no_connect
 		(at 168.91 57.15)
 	)
+	(no_connect
+		(at 181.61 111.76)
+	)
+	(no_connect
+		(at 194.31 111.76)
+	)
+	(no_connect
+		(at 191.77 147.32)
+	)
+	(no_connect
+		(at 199.39 147.32)
+	)
+	(no_connect
+		(at 179.07 147.32)
+	)
 	(wire

Commit message: PCB Layout V2
Parts:
- added C19: 100 nF, Capacitor_SMD_Wurth:C_Wurth_WCAP-CSGP-1206_H0.8, symbol symbols:1206_H0.8_885012208030
Connections:
- net GND: now also C19.2
- net NRST: now also C19.1
Other:
- moved on the sheet: SW1

Commit message: Update PCB mit GND Plane
Parts:
- added TP1: TP_TX_A, TestPoint:TestPoint_Pad_D2.0mm, symbol Connector:TestPoint
- added TP11: TP_3_3V, TestPoint:TestPoint_Pad_D2.0mm, symbol Connector:TestPoint
- added TP12: TP_5V, TestPoint:TestPoint_Pad_D2.0mm, symbol Connector:TestPoint
- added TP13: TP_GND_2, TestPoint:TestPoint_Pad_D2.0mm, symbol Connector:TestPoint
- added TP14: TP_X_Axis, TestPoint:TestPoint_Pad_D2.0mm, symbol Connector:TestPoint
- added TP15: TP_Y_Axis, TestPoint:TestPoint_Pad_D2.0mm, symbol Connector:TestPoint
- added TP16: TP_Z_Axis, TestPoint:TestPoint_Pad_D2.0mm, symbol Connector:TestPoint
- added TP2: TP_RX_A, TestPoint:TestPoint_Pad_D2.0mm, symbol Connector:TestPoint
- added TP3: TP_DE_A, TestPoint:TestPoint_Pad_D2.0mm, symbol Connector:TestPoint
- added TP4: TP_NRE_A, TestPoint:TestPoint_Pad_D2.0mm, symbol Connector:TestPoint
- added TP5: TP_TX_B, TestPoint:TestPoint_Pad_D2.0mm, symbol Connector:TestPoint
- added TP6: TP_RX_B, TestPoint:TestPoint_Pad_D2.0mm, symbol Connector:TestPoint
- added TP7: TP_DE_B, TestPoint:TestPoint_Pad_D2.0mm, symbol Connector:TestPoint
- added TP8: TP_NRE_B, TestPoint:TestPoint_Pad_D2.0mm, symbol Connector:TestPoint
- added TP9: TP_GND_1, TestPoint:TestPoint_Pad_D2.0mm, symbol Connector:TestPoint
Connections:
- net GND: now also TP13.1, TP9.1
- net JS_X_axis: now also TP14.1
- net JS_Y_axis: now also TP15.1
- net JS_Z_axis: now also TP16.1
- net UART_DE_Mtr_A: now also TP3.1
- net UART_DE_Mtr_B: now also TP7.1
- net UART_NRE_Mtr_A: now also TP4.1
- net UART_NRE_Mtr_B: now also TP8.1
- net UART_RX_Mtr_A: now also TP2.1
- net UART_RX_Mtr_B: now also TP6.1
- net UART_TX_Mtr_A: now also TP1.1
- net UART_TX_Mtr_B: now also TP5.1
- net VCC_3_3V: now also TP11.1
- net VCC_5V: now also TP12.1
Other:
- moved on the sheet: R5, U3

Commit message: Final Changes
Finale Aenderung am PCB Erzeugung der Drill und Gerber Files
Parts:
- added H1, H2, H3: MountingHole, MountingHole:MountingHole_3.2mm_M3, symbol Mechanical:MountingHole
Changed lines of the file:
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@@
 	)
 	(symbol
+		(lib_id "Mechanical:MountingHole")
+		(at 266.7 105.41 0)
+		(unit 1)
+		(body_style 1)
+		(exclude_from_sim no)
+		(in_bom no)
+		(on_board yes)
+		(in_pos_files yes)
+		(dnp no)
+		(fields_autoplaced yes)
+		(property "Reference" "H3"
+			(at 269.24 104.1399 0)
+			(show_name no)
+			(do_not_autoplace no)
+			(effects
+				(font
+					(size 1.27 1.27)
+				)
+				(justify left)
+			)
+		)
+		(property "Value" "MountingHole"
+			(at 269.24 106.6799 0)
+			(show_name no)
+			(do_not_autoplace no)
+			(effects
+				(font
+					(size 1.27 1.27)
+				)
+				(justify left)
+			)
+		)
+		(property "Footprint" "MountingHole:MountingHole_3.2mm_M3"
+			(at 266.7 105.41 0)
+			(hide yes)
+			(show_name no)
+			(do_not_autoplace no)
+			(effects
+				(font
+					(size 1.27 1.27)
+				)
+			)
+		)
+		(property "Datasheet" ""
+			(at 266.7 105.41 0)
+			(hide yes)
+			(show_name no)
+			(do_not_autoplace no)
+			(effects
+				(font
+					(size 1.27 1.27)
+				)
+			)
+		)
+		(property "Description" "Mounting Hole without connection"
+			(at 266.7 105.41 0)
+			(hide yes)
+			(show_name no)
+			(do_not_autoplace no)
+			(effects
+				(font
+					(size 1.27 1.27)
+				)
+			)
+		)
+		(instances
+			(project "KommModul_Joystick"
+				(path "/b3a1d19e-72ec-433f-985d-69e9858988ab"
+					(reference "H3")
+					(unit 1)
+				)
+			)
+		)
+	)
+	(symbol
 		(lib_id "symbols:1206_R_560112132038")
 		(at 43.18 24.13 270)
@@
 	)
 	(symbol
+		(lib_id "Mechanical:MountingHole")
+		(at 266.7 83.82 0)
+		(unit 1)
+		(body_style 1)
+		(exclude_from_sim no)
+		(in_bom no)
+		(on_board yes)
+		(in_pos_files yes)
+		(dnp no)
+		(fields_autoplaced yes)
+		(property "Reference" "H1"
+			(at 269.24 82.5499 0)
+			(show_name no)
+			(do_not_autoplace no)
+			(effects
+				(font
+					(size 1.27 1.27)
+				)
+				(justify left)
+			)
+		)
+		(property "Value" "MountingHole"
+			(at 269.24 85.0899 0)
+			(show_name no)
+			(do_not_autoplace no)
+			(effects
+				(font
+					(size 1.27 1.27)
+				)
+				(justify left)
+			)
+		)
+		(property "Footprint" "MountingHole:MountingHole_3.2mm_M3"
+			(at 266.7 83.82 0)
+			(hide yes)
+			(show_name no)
+			(do_not_autoplace no)
+			(effects
+				(font
+					(size 1.27 1.27)
+				)
+			)
+		)
+		(property "Datasheet" ""
+			(at 266.7 83.82 0)
+			(hide yes)
+			(show_name no)
+			(do_not_autoplace no)
+			(effects
+				(font
+					(size 1.27 1.27)
+				)
+			)
+		)
+		(property "Description" "Mounting Hole without connection"
+			(at 266.7 83.82 0)
+			(hide yes)
+			(show_name no)
+			(do_not_autoplace no)
+			(effects
+				(font
+					(size 1.27 1.27)
+				)
+			)
+		)
+		(instances
+			(project "KommModul_Joystick"
+				(path "/b3a1d19e-72ec-433f-985d-69e9858988ab"
+					(reference "H1")
+					(unit 1)
+				)
+			)
+		)
+	)
+	(symbol
 		(lib_id "Connector:TestPoint")
 		(at 115.57 35.56 0)
@@
 					(unit 1)
 				)
+			)
+		)
+	)
+	(symbol
+		(lib_id "Mechanical:MountingHole")
+		(at 266.7 93.98 0)
+		(unit 1)
+		(body_style 1)
+		(exclude_from_sim no)
+		(in_bom no)
+		(on_board yes)
+		(in_pos_files yes)
+		(dnp no)
+		(fields_autoplaced yes)
+		(property "Reference" "H2"
+			(at 269.24 92.7099 0)
+			(show_name no)
+			(do_not_autoplace no)
+			(effects
+				(font
+					(size 1.27 1.27)
+				)
+				(justify left)
+			)
+		)
+		(property "Value" "MountingHole"
+			(at 269.24 95.2499 0)
+			(show_name no)
+			(do_not_autoplace no)
+			(effects
+				(font
+					(size 1.27 1.27)
+				)
+				(justify left)
+			)
+		)
+		(property "Footprint" "MountingHole:MountingHole_3.2mm_M3"
+			(at 266.7 93.98 0)
+			(hide yes)
+			(show_name no)
+			(do_not_autoplace no)
+			(effects
+				(font
+					(size 1.27 1.27)
+				)
+			)
+		)
+		(property "Datasheet" ""
+			(at 266.7 93.98 0)
+			(hide yes)
+			(show_name no)
+			(do_not_autoplace no)
+			(effects
+				(font
+					(size 1.27 1.27)
+				)
+			)
+		)
+		(property "Description" "Mounting Hole without connection"
+			(at 266.7 93.98 0)
+			(hide yes)
+			(show_name no)
+			(do_not_autoplace no)
+			(effects
+				(font
+					(size 1.27 1.27)
+				)
+			)
+		)
+		(instances
+			(project "KommModul_Joystick"
+				(path "/b3a1d19e-72ec-433f-985d-69e9858988ab"
+					(reference "H2")
+					(unit 1)
+				)
